Commit message: Fix controller loop

File: urdf/diff_drive_description.xacro (robot description, xacro)
@@ -1,5 +1,187 @@
 <?xml version="1.0" encoding="UTF-8" ?>
-<robot name="mock_robot" xmlns:xacro="http://www.ros.org/wiki/xacro">
-  <!-- The robot link description -->
-  <link name="base_link" />
+<robot name="Bumbar" xmlns:xacro="http://www.ros.org/wiki/xacro" >
+    <xacro:include filename="inertial_macros.xacro"/>
+    <xacro:include filename="camera.xacro"/>
+    <xacro:include filename="lidar.xacro"/>
+    <xacro:property name="chassis_length" value="0.20"/>
+    <xacro:property name="chassis_width" value="0.16"/>
+    <xacro:property name="chassis_height" value="0.26"/>
+    <xacro:property name="chassis_mass" value="1.0"/>
+    <xacro:property name="wheel_radius" value="0.039"/>
+    <xacro:property name="wheel_thickness" value="0.041"/>
+    <xacro:property name="wheel_mass" value="0.05"/>
+    <!-- FRONT LEFT WHEEL -->
+    <xacro:property name="front_left_wheel_offset_x" value="-0.1"/>
+    <xacro:property name="front_left_wheel_offset_y" value="0.05"/>
+    <xacro:property name="front_left_wheel_offset_z" value="0.01"/>
+    <!-- FRONT RIGHT WHEEL -->
+    <xacro:property name="front_right_wheel_offset_x" value="0.10"/>
+    <xacro:property name="front_right_wheel_offset_y" value="0.05"/>
+    <xacro:property name="front_right_wheel_offset_z" value="0.01"/>
+    <!-- BACK LEFT WHEEL -->
+    <xacro:property name="bacK_left_wheel_offset_x" value="-0.1"/>
+    <xacro:property name="bacK_left_wheel_offset_y" value="-0.05"/>
+    <xacro:property name="bacK_left_wheel_offset_z" value="0.01"/>
+    <!-- BACK RIGHT WHEEL -->
+    <xacro:property name="bacK_right_wheel_offset_x" value="0.1"/>
+    <xacro:property name="bacK_right_wheel_offset_y" value="-0.05"/>
+    <xacro:property name="bacK_right_wheel_offset_z" value="0.01"/>
+    <material name="white">
+        <color rgba="1 1 1 1" />
+    </material>
+    <material name="orange">
+        <color rgba="1 0.3 0.1 1"/>
+    </material>
+    <material name="blue">
+        <color rgba="0.2 0.2 1 1"/>
+    </material>
+    <material name="black">
+        <color rgba="0 0 0 1"/>
+    </material>
+    <material name="red">
+        <color rgba="1 0 0 1"/>
+    </material>
+    <!-- BASE LINK -->
+    <link name="base_link">
+    </link>
+    <!-- CHASSIS LINK -->
+    <joint name="chassis_joint" type="fixed">
+        <parent link="base_link"/>
+        <child link="chassis"/>
+        <!-- <origin xyz="${-wheel_offset_x} 0 ${-wheel_offset_z}"/> -->
+        <origin xyz="0.0 0.0 0.1739"/>
+    </joint>
+    <link name="chassis">
+        <visual>
+            <origin xyz="0.0 0.0 0.0"/>
+            <geometry>
+                <box size="${chassis_length} ${chassis_width} ${chassis_height}"/>
+            </geometry>
+            <material name="orange"/>
+        </visual>
+        <collision>
+            <origin xyz="0.0 0 0.0"/>
+            <geometry>
+                <box size="${chassis_length} ${chassis_width} ${chassis_height}"/>
+            </geometry>
+        </collision>
+        <xacro:inertial_box mass="0.5" x="${chassis_length}" y="${chassis_width}" z="${chassis_height}">
+            <origin xyz="0.1 0 0.14" rpy="0 0 0"/>
+        </xacro:inertial_box>
+    </link>
+    <gazebo reference="chassis">
+        <material>Gazebo/Orange</material>
+    </gazebo>
+    <!--FRONT RIGHT WHEEL LINK -->
+    <joint name="front_right_wheel_joint" type="continuous">
+        <parent link="base_link"/>
+        <child link="front_right_wheel"/>
+        <origin xyz="0.05 -0.1  0.039" rpy="${pi/2} 0 0" />
+        <axis xyz="0 0 -1"/>
+    </joint>
+    <link name="front_right_wheel">
+        <visual>
+            <geometry>
+                <cylinder radius="${wheel_radius}" length="${wheel_thickness}"/>
+            </geometry>
+            <material name="blue"/>
+        </visual>
+        <collision>
+            <geometry>
+                <sphere radius="${wheel_radius}"/>
+            </geometry>
+            <origin xyz="0.0 0  0" rpy="${pi/2} 0 0" />
+            <!--axis xyz="0 -1 -1"/-->
+        </collision>
+        <xacro:inertial_cylinder mass="${wheel_mass}" length="${wheel_thickness}" radius="${wheel_radius}">
+           <origin xyz="0.0 0  0.0" rpy="${pi/2} 0 0" />
+            <!--axis xyz="0 -1 -1"/-->
+        </xacro:inertial_cylinder>
+    </link>
+    <gazebo reference="front_right_wheel">
+        <material>Gazebo/Blue</material>
+    </gazebo>
+    <!-- FRONT RIGHT WHEEL LINK -->
+    <joint name="fron_left_wheel_joint" type="continuous">
+        <parent link="base_link"/>
+        <child link="front_left_wheel"/>
+        <origin xyz="0.05 0.1 0.039" rpy="-${pi/2} 0 0" />
+        <axis xyz="0 0 1"/>
+    </joint>
+    <link name="front_left_wheel">
+        <visual>
+            <geometry>
+                <cylinder radius="${wheel_radius}" length="${wheel_thickness}"/>
+            </geometry>
+            <material name="blue"/>
+        </visual>
+        <collision>
+            <geometry>
+                <sphere radius="${wheel_radius}"/>
+            </geometry>
+        </collision>
+        <xacro:inertial_cylinder mass="${wheel_mass}" length="${wheel_thickness}" radius="${wheel_radius}">
+            <origin xyz="0.0 0 0.0" rpy="-${pi/2} 0 0" />
+            <!--axis xyz="0 1 1"/-->
+        </xacro:inertial_cylinder>
+    </link>
+    <gazebo reference="front_right_wheel">
+        <material>Gazebo/Blue</material>
+    </gazebo>
+    <!-- BACK RIGHT WHEEL LINK -->
+    <joint name="back_right_wheel_joint" type="continuous">
+        <parent link="base_link"/>
+        <child link="back_right_wheel"/>
+        <origin xyz="-0.05 -0.1  0.039" rpy="${pi/2} 0 0" />
+        <axis xyz="0 0 -1"/>
+    </joint>
+    <link name="back_right_wheel">
+        <visual>
+            <geometry>
+                <cylinder radius="${wheel_radius}" length="${wheel_thickness}"/>
+            </geometry>
+            <material name="blue"/>
+        </visual>
+        <collision>
+            <geometry>
+                <sphere radius="${wheel_radius}"/>
+            </geometry>
+            <origin xyz="0.0 0  0.0" rpy="${pi/2} 0 0" />
+            <!--axis xyz="0 0 -1"/-->
+        </collision>
+        <xacro:inertial_cylinder mass="${wheel_mass}" length="${wheel_thickness}" radius="${wheel_radius}">
+            <origin xyz="0.0 0  0.0" rpy="${pi/2} 0 0" />
+        </xacro:inertial_cylinder>
+    </link>
+    <gazebo reference="back_right_wheel">
+        <material>Gazebo/Blue</material>
+    </gazebo>
+    <!-- BACK LEFT WHEEL LINK -->
+    <joint name="back_left_wheel_joint" type="continuous">
+        <parent link="base_link"/>
+        <child link="back_left_wheel"/>
+        <origin xyz="-0.05 0.1 0.039" rpy="-${pi/2} 0 0" />
+        <axis xyz="0 0 1"/>
+    </joint>
+    <link name="back_left_wheel">
+        <visual>
+            <geometry>
+                <cylinder radius="${wheel_radius}" length="${wheel_thickness}"/>
+            </geometry>
+            <material name="blue"/>
+        </visual>
+        <collision>
+            <geometry>
+                <sphere radius="${wheel_radius}"/>
+            </geometry>
+            <origin xyz="0.0 0. 0.0" rpy="-${pi/2} 0 0" />
+            <!--axis xyz="0 0 1"/-->
+        </collision>
+        <xacro:inertial_cylinder mass="${wheel_mass}" length="${wheel_thickness}" radius="${wheel_radius}">
+            <origin xyz="0.0 0 0.0" rpy="-${pi/2} 0 0" />
+        </xacro:inertial_cylinder>
+    </link>
+    <gazebo reference="left_wheel">
+        <material>Gazebo/Blue</material>
+    </gazebo>
 </robot>
